File: weather_station_pico.kicad_pcb (KiCad board)
At the start: 2 copper layers, 88.5 x 90 mm, 30 parts, among them J1 POWER, J2 WSPEED, J3 WDIR, J4 I2C, SW1 SW_Push, U1 LM7805_TO220, U2 E220-900T22D, U3 Pico, U4 74HC4051, U5 LM35-LP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

Commit message: add millproject
Parts:
- removed TP1: TEMP_REF, TestPoint:TestPoint_Pad_D1.5mm
- removed TP2: GND, TestPoint:TestPoint_Pad_D1.5mm
- removed TP3: TEMP_OUT, TestPoint:TestPoint_Pad_D1.5mm
- removed TP4: MUX_ADC, TestPoint:TestPoint_Pad_D1.5mm
- moved SW1 9.11 mm to (176.5, 73.0), turned to 0 degrees
- moved R6 5.08 mm to (128.3, 108.2)
- moved U6 2.97 mm to (147.3, 108.0), turned to 180 degrees
- moved R10 2.54 mm to (132.1, 108.2)
- moved R3 1.98 mm to (171.4, 118.4)
- moved R4 1.98 mm to (175.3, 108.2)
- moved U1 1.31 mm to (185.4, 59.7)
- moved U5 0.19 mm to (141.0, 114.3)
Connections:
- U3 pad 42: GND -> unconnected-(U3-Pad42)
Routing:
- net +3V3: track 122.1 -> 155.2 mm, vias 3 -> 2
- net /SDA: track 53.4 -> 83.9 mm
- net +5V: track 91.5 -> 113.6 mm, vias 1 -> 0
- net /SCL: track 59.6 -> 80.7 mm
- net +12V: track 122.9 -> 141.5 mm
- net /IN_TEMP_REF: track 54.0 -> 46.0 mm
- net /IN_TEMP_OUT: track 53.4 -> 46.3 mm
- net /LORA_AUX: track 31.9 -> 37.9 mm
- net /RUN: track 18.5 -> 13.4 mm
- net /LORA_TXD: track 28.9 -> 32.6 mm, vias 1 -> 0
- net /MUX_EN: track 20.9 -> 23.9 mm, vias 1 -> 0
- net /MUX_ADC: track 44.5 -> 46.8 mm
- net /LORA_RXD: track 24.7 -> 26.2 mm, vias 0 -> 2
- net /WDIR_5V: track 7.62 -> 8.44 mm
- removed copper zone on F.Cu, net GND
